File: rapid_sensor_board.kicad_sch (KiCad schematic)
At the start: 43 parts, among them IC1 INA826AID, J1 JST-GH, J2 JST-GH, J3 Conn_01x02_Socket, J5 Conn_01x04_Socket, U2 MCP6001-OT, U3 MIC5504-3.3YM5, U4 ADC101C021CIMM

Commit message: some changes, added production files
Parts:
- added TP1: TestPoint, TestPoint:TestPoint_Pad_D1.5mm, symbol Connector:TestPoint
- C1: LCSC C315248 -> C15525
- C10, C9: value 2n2 -> 1n; LCSC C84703 -> C1523
- C15, C16: LCSC C76999 -> C52923
- D2, D3, D7, D8: LCSC C48935658 -> C20933
- D4: LCSC (none) -> C20933
- IC1: LCSC C38433 -> C2870890
- J1, J2, R3, R7, R8, RG1: now not fitted
- R10, R9: LCSC (none) -> C25076; LCSC# C106232 -> (none); Manufacturer YAGEO -> (none); Part# RC0402FR-07100RL -> (none)
- U4: footprint Package_SO:MSOP-8_3x3mm_P0.65mm -> Package_SO:VSSOP-8_3x3mm_P0.65mm
Connections:
- net 3V3: now also R3.1, TP1.1; no longer J3.2 (Pin_2), R4.1
- net GND: now also J3.1 (Pin_1), R4.2; no longer R3.2
- net s+: now also J3.2 (Pin_2), R3.2, R4.1; no longer J3.1 (Pin_1), R3.1, R4.2
Other:
- note added: "1n chosen as 2n2 not a basic part"
- note added: "TUDSaT Sensor Board"
- note removed: "TUDSaT Amplifier Board"
- moved on the sheet: J3, R4
